Commit message: add pt

File: rasberrypi/catkin_ws/src/humanoid_urdf_description/urdf/humanoid_urdf.urdf (robot description, URDF)
Before this commit: robot humanoid_urdf, 33 links, 32 joints
Joints:
- removed joint ll2_joint
- added joint ȸ�� 123: type revolute, parent ll2_1, child ll3_1, origin xyz=-0.01825 0.019 -8e-06 rpy=0 0 0, axis -0.0 1.0 -0.0, limit lower=-1.570796 upper=0.349066 effort=100 velocity=100
- joint lelbow_joint: axis 0.0 0.0 -1.0 -> 0.0 -0.996195 -0.087156; origin xyz=0.0 0.0437 -0.019 rpy=0 0 0 -> xyz=0.0 -0.015119 -0.04519 rpy=0 0 0
- joint lgrip_fin1_slider: axis 1.0 0.0 0.0 -> 1.0 0.0 -0.0; limit lower=-0.02 upper=0.007 effort=100 velocity=100 -> lower=0.0 upper=0.0 effort=100 velocity=100; mimic joint=lgripper_joint multiplier=0.00869 offset=0.0 -> (none); origin xyz=0.018907 0.0389 0.0192 rpy=0 0 0 -> xyz=0.018907 0.022518 -0.037079 rpy=0 0 0
- joint lgrip_fin2_slider: axis 1.0 0.0 0.0 -> 1.0 0.0 -0.0; limit lower=-0.007 upper=0.02 effort=100 velocity=100 -> lower=0.0 upper=0.0 effort=100 velocity=100; mimic joint=lgrip_fin1_slider multiplier=-1.0 offset=0.0 -> (none); origin xyz=0.019 0.0389 -0.0192 rpy=0 0 0 -> xyz=0.019 -0.015736 -0.040425 rpy=0 0 0
- joint lgripper_joint: axis -0.0 1.0 0.0 -> -0.0 0.087156 -0.996195; limit lower=-5.2360 upper=0.8727 effort=100 velocity=100 -> lower=-1.745329 upper=0.261799 effort=100 velocity=100; origin xyz=0.019 0.0397 0.0 rpy=0 0 0 -> xyz=0.019 0.00346 -0.039549 rpy=0 0 0
- joint ll3_joint: origin xyz=-6.5e-05 0.0 -0.087294 rpy=0 0 0 -> xyz=0.0 -0.0356 -0.092493 rpy=0 0 0
- joint ll4_joint: origin xyz=0.0 0.0 -0.092485 rpy=0 0 0 -> xyz=0.0 0.0 -0.092486 rpy=0 0 0
- joint lshd_pitch_joint: limit lower=-3.141592 upper=3.141592 effort=100 velocity=100 -> lower=-1.570796 upper=1.570796 effort=100 velocity=100
- joint lshd_roll_joint: axis -0.0 1.0 0.0 -> -0.0 0.087156 -0.996195; origin xyz=0.019 0.026 0.0 rpy=0 0 0 -> xyz=0.019 0.002266 -0.025901 rpy=0 0 0
- joint lshd_yaw_joint: limit lower=-1.570796 upper=0.349066 effort=100 velocity=100 -> lower=-0.349066 upper=1.570796 effort=100 velocity=100
- joint lwrist_pitch_joint: axis 0.0 0.0 -1.0 -> 0.0 -0.996195 -0.087156; origin xyz=0.0 0.1002 0.045 rpy=0 0 0 -> xyz=0.0 0.053562 -0.095897 rpy=0 0 0
- joint lwrist_yaw_joint: axis -1.0 -0.0 -0.0 -> -1.0 -0.0 0.0; origin xyz=-0.019 0.0 -0.0287 rpy=0 0 0 -> xyz=-0.019 -0.028591 -0.002501 rpy=0 0 0
- joint relbow_joint: axis -0.0 -0.0 -1.0 -> -0.0 0.996195 -0.087156; origin xyz=0.0 -0.0437 -0.019 rpy=0 0 0 -> xyz=0.0 0.015119 -0.04519 rpy=0 0 0
- joint rgrip_fin1_slider: limit lower=-0.02 upper=0.007 effort=100 velocity=100 -> lower=0.0 upper=0.0 effort=100 velocity=100; mimic joint=rgripper_joint multiplier=0.00869 offset=0.0 -> (none); origin xyz=-0.019 -0.0389 -0.0192 rpy=0 0 0 -> xyz=-0.019 0.015737 -0.040425 rpy=0 0 0
- joint rgrip_fin2_slider: limit lower=-0.007 upper=0.02 effort=100 velocity=100 -> lower=0.0 upper=0.0 effort=100 velocity=100; mimic joint=rgrip_fin1_slider multiplier=-1.0 offset=0.0 -> (none); origin xyz=-0.019093 -0.0389 0.0192 rpy=0 0 0 -> xyz=-0.019093 -0.022517 -0.037079 rpy=0 0 0
- joint rgripper_joint: axis -0.0 1.0 0.0 -> -0.0 0.087156 0.996195; limit lower=-5.2360 upper=0.8727 effort=100 velocity=100 -> lower=-1.745329 upper=0.261799 effort=100 velocity=100; origin xyz=-0.019 -0.0397 0.0 rpy=0 0 0 -> xyz=-0.019 -0.00346 -0.039549 rpy=0 0 0
- joint rshd_pitch_joint: limit lower=-3.141592 upper=3.141592 effort=100 velocity=100 -> lower=-1.570796 upper=1.570796 effort=100 velocity=100
- joint rshd_roll_joint: axis 0.0 -1.0 0.0 -> 0.0 -0.087156 -0.996195; origin xyz=0.018 -0.026 0.0 rpy=0 0 0 -> xyz=0.018 -0.002266 -0.025901 rpy=0 0 0
- joint rshd_yaw_joint: limit lower=-0.349066 upper=1.570796 effort=100 velocity=100 -> lower=-1.570796 upper=0.0 effort=100 velocity=100
- joint rwrist_pitch_joint: axis 0.0 -0.0 -1.0 -> 0.0 0.996195 -0.087156; origin xyz=0.0 -0.1002 0.045 rpy=0 0 0 -> xyz=0.0 -0.053562 -0.095897 rpy=0 0 0
- joint rwrist_yaw_joint: axis 1.0 0.0 0.0 -> 1.0 -0.0 0.0; origin xyz=0.019 0.0 -0.0287 rpy=0 0 0 -> xyz=0.019 0.028591 -0.002501 rpy=0 0 0

File: rasberrypi/catkin_ws/src/opencr_rcm_control/urdf/humanoid.urdf (robot description, URDF)
Before this commit: robot humanoid_urdf, 33 links, 32 joints
Joints:
- joint lelbow_joint: axis 0.0 0.0 -1.0 -> 0.0 -0.996195 -0.087156; origin xyz=0.0 0.0437 -0.019 rpy=0 0 0 -> xyz=0.0 -0.015119 -0.04519 rpy=0 0 0
- joint lgripper_joint: axis -0.0 1.0 0.0 -> -0.0 0.087156 -0.996195; limit lower=-5.2360 upper=0.8727 effort=100 velocity=100 -> lower=-1.745329 upper=0.261799 effort=100 velocity=100; origin xyz=0.019 0.0397 0.0 rpy=0 0 0 -> xyz=0.019 0.00346 -0.039549 rpy=0 0 0
- joint ll2_joint: axis 0.0 -1.0 0.0 -> -0.0 1.0 -0.0; limit lower=-0.349066 upper=1.570796 effort=100 velocity=100 -> lower=-1.570796 upper=0.349066 effort=100 velocity=100; origin xyz=-0.01825 -0.019 -8e-06 rpy=0 0 0 -> xyz=-0.01825 0.019 -8e-06 rpy=0 0 0
- joint ll3_joint: origin xyz=-6.5e-05 0.0 -0.087294 rpy=0 0 0 -> xyz=0.0 -0.0356 -0.092493 rpy=0 0 0
- joint ll4_joint: origin xyz=0.0 0.0 -0.092485 rpy=0 0 0 -> xyz=0.0 0.0 -0.092486 rpy=0 0 0
- joint lshd_pitch_joint: limit lower=-3.141592 upper=3.141592 effort=100 velocity=100 -> lower=-1.570796 upper=1.570796 effort=100 velocity=100
- joint lshd_roll_joint: axis -0.0 1.0 0.0 -> -0.0 0.087156 -0.996195; origin xyz=0.019 0.026 0.0 rpy=0 0 0 -> xyz=0.019 0.002266 -0.025901 rpy=0 0 0
- joint lshd_yaw_joint: limit lower=-1.570796 upper=0.349066 effort=100 velocity=100 -> lower=0.0 upper=1.570796 effort=100 velocity=100
- joint lwrist_pitch_joint: axis 0.0 0.0 -1.0 -> 0.0 -0.996195 -0.087156; origin xyz=0.0 0.1002 0.045 rpy=0 0 0 -> xyz=0.0 0.053562 -0.095897 rpy=0 0 0
- joint lwrist_yaw_joint: axis -1.0 -0.0 -0.0 -> -1.0 -0.0 0.0; origin xyz=-0.019 0.0 -0.0287 rpy=0 0 0 -> xyz=-0.019 -0.028591 -0.002501 rpy=0 0 0
- joint relbow_joint: axis -0.0 -0.0 -1.0 -> -0.0 0.996195 -0.087156; origin xyz=0.0 -0.0437 -0.019 rpy=0 0 0 -> xyz=0.0 0.015119 -0.04519 rpy=0 0 0
- joint rgripper_joint: axis -0.0 1.0 0.0 -> -0.0 0.087156 0.996195; limit lower=-5.2360 upper=0.8727 effort=100 velocity=100 -> lower=-1.745329 upper=0.261799 effort=100 velocity=100; origin xyz=-0.019 -0.0397 0.0 rpy=0 0 0 -> xyz=-0.019 -0.00346 -0.039549 rpy=0 0 0
- joint rshd_pitch_joint: limit lower=-3.141592 upper=3.141592 effort=100 velocity=100 -> lower=-1.570796 upper=1.570796 effort=100 velocity=100
- joint rshd_roll_joint: axis 0.0 -1.0 0.0 -> 0.0 -0.087156 -0.996195; origin xyz=0.018 -0.026 0.0 rpy=0 0 0 -> xyz=0.018 -0.002266 -0.025901 rpy=0 0 0
- joint rshd_yaw_joint: limit lower=-0.349066 upper=1.570796 effort=100 velocity=100 -> lower=0.0 upper=1.570796 effort=100 velocity=100
- joint rwrist_pitch_joint: axis 0.0 -0.0 -1.0 -> 0.0 0.996195 -0.087156; origin xyz=0.0 -0.1002 0.045 rpy=0 0 0 -> xyz=0.0 -0.053562 -0.095897 rpy=0 0 0
- joint rwrist_yaw_joint: axis 1.0 0.0 0.0 -> 1.0 -0.0 0.0; origin xyz=0.019 0.0 -0.0287 rpy=0 0 0 -> xyz=0.019 0.028591 -0.002501 rpy=0 0 0

File: train_arm/humanoid_urdf_description/urdf/humanoid_urdf.urdf (robot description, URDF)
Before this commit: robot humanoid_urdf, 33 links, 32 joints
Joints:
- joint lelbow_joint: axis 0.0 0.0 -1.0 -> 0.0 -0.996195 -0.087156; origin xyz=0.0 0.0437 -0.019 rpy=0 0 0 -> xyz=0.0 -0.015119 -0.04519 rpy=0 0 0
- joint lgrip_fin1_slider: axis 1.0 0.0 0.0 -> 1.0 0.0 -0.0; limit lower=-0.02 upper=0.007 effort=100 velocity=100 -> lower=0.0 upper=0.0 effort=100 velocity=100; mimic joint=lgripper_joint multiplier=0.00869 offset=0.0 -> (none); origin xyz=0.018907 0.0389 0.0192 rpy=0 0 0 -> xyz=0.018907 0.022518 -0.037079 rpy=0 0 0
- joint lgrip_fin2_slider: axis 1.0 0.0 0.0 -> 1.0 0.0 -0.0; limit lower=-0.007 upper=0.02 effort=100 velocity=100 -> lower=0.0 upper=0.0 effort=100 velocity=100; mimic joint=lgrip_fin1_slider multiplier=-1.0 offset=0.0 -> (none); origin xyz=0.019 0.0389 -0.0192 rpy=0 0 0 -> xyz=0.019 -0.015736 -0.040425 rpy=0 0 0
- joint lgripper_joint: axis -0.0 1.0 0.0 -> -0.0 0.087156 -0.996195; limit lower=-5.2360 upper=0.8727 effort=100 velocity=100 -> lower=-1.745329 upper=0.261799 effort=100 velocity=100; origin xyz=0.019 0.0397 0.0 rpy=0 0 0 -> xyz=0.019 0.00346 -0.039549 rpy=0 0 0
- joint ll2_joint: axis 0.0 -1.0 0.0 -> -0.0 1.0 -0.0; limit lower=-0.349066 upper=1.570796 effort=100 velocity=100 -> lower=-1.570796 upper=0.349066 effort=100 velocity=100; origin xyz=-0.01825 -0.019 -8e-06 rpy=0 0 0 -> xyz=-0.01825 0.019 -8e-06 rpy=0 0 0
- joint ll3_joint: origin xyz=-6.5e-05 0.0 -0.087294 rpy=0 0 0 -> xyz=0.0 -0.0356 -0.092493 rpy=0 0 0
- joint ll4_joint: origin xyz=0.0 0.0 -0.092485 rpy=0 0 0 -> xyz=0.0 0.0 -0.092486 rpy=0 0 0
- joint lshd_pitch_joint: limit lower=-3.141592 upper=3.141592 effort=100 velocity=100 -> lower=-1.570796 upper=1.570796 effort=100 velocity=100
- joint lshd_roll_joint: axis -0.0 1.0 0.0 -> -0.0 0.087156 -0.996195; origin xyz=0.019 0.026 0.0 rpy=0 0 0 -> xyz=0.019 0.002266 -0.025901 rpy=0 0 0
- joint lshd_yaw_joint: limit lower=-1.570796 upper=0.349066 effort=100 velocity=100 -> lower=-0.349066 upper=1.570796 effort=100 velocity=100
- joint lwrist_pitch_joint: axis 0.0 0.0 -1.0 -> 0.0 -0.996195 -0.087156; origin xyz=0.0 0.1002 0.045 rpy=0 0 0 -> xyz=0.0 0.053562 -0.095897 rpy=0 0 0
- joint lwrist_yaw_joint: axis -1.0 -0.0 -0.0 -> -1.0 -0.0 0.0; origin xyz=-0.019 0.0 -0.0287 rpy=0 0 0 -> xyz=-0.019 -0.028591 -0.002501 rpy=0 0 0
- joint relbow_joint: axis -0.0 -0.0 -1.0 -> -0.0 0.996195 -0.087156; origin xyz=0.0 -0.0437 -0.019 rpy=0 0 0 -> xyz=0.0 0.015119 -0.04519 rpy=0 0 0
- joint rgrip_fin1_slider: limit lower=-0.02 upper=0.007 effort=100 velocity=100 -> lower=0.0 upper=0.0 effort=100 velocity=100; mimic joint=rgripper_joint multiplier=0.00869 offset=0.0 -> (none); origin xyz=-0.019 -0.0389 -0.0192 rpy=0 0 0 -> xyz=-0.019 0.015737 -0.040425 rpy=0 0 0
- joint rgrip_fin2_slider: limit lower=-0.007 upper=0.02 effort=100 velocity=100 -> lower=0.0 upper=0.0 effort=100 velocity=100; mimic joint=rgrip_fin1_slider multiplier=-1.0 offset=0.0 -> (none); origin xyz=-0.019093 -0.0389 0.0192 rpy=0 0 0 -> xyz=-0.019093 -0.022517 -0.037079 rpy=0 0 0
- joint rgripper_joint: axis -0.0 1.0 0.0 -> -0.0 0.087156 0.996195; limit lower=-5.2360 upper=0.8727 effort=100 velocity=100 -> lower=-1.745329 upper=0.261799 effort=100 velocity=100; origin xyz=-0.019 -0.0397 0.0 rpy=0 0 0 -> xyz=-0.019 -0.00346 -0.039549 rpy=0 0 0
- joint rshd_pitch_joint: limit lower=-3.141592 upper=3.141592 effort=100 velocity=100 -> lower=-1.570796 upper=1.570796 effort=100 velocity=100
- joint rshd_roll_joint: axis 0.0 -1.0 0.0 -> 0.0 -0.087156 -0.996195; origin xyz=0.018 -0.026 0.0 rpy=0 0 0 -> xyz=0.018 -0.002266 -0.025901 rpy=0 0 0
- joint rshd_yaw_joint: limit lower=-0.349066 upper=1.570796 effort=100 velocity=100 -> lower=-1.570796 upper=0.0 effort=100 velocity=100
- joint rwrist_pitch_joint: axis 0.0 -0.0 -1.0 -> 0.0 0.996195 -0.087156; origin xyz=0.0 -0.1002 0.045 rpy=0 0 0 -> xyz=0.0 -0.053562 -0.095897 rpy=0 0 0
- joint rwrist_yaw_joint: axis 1.0 0.0 0.0 -> 1.0 -0.0 0.0; origin xyz=0.019 0.0 -0.0287 rpy=0 0 0 -> xyz=0.019 0.028591 -0.002501 rpy=0 0 0
